File: Brakeman.brd (EAGLE design)
At the start: 25.3 x 34.5 mm, 11 parts

Commit message: 1.0
Parts:
- removed PAD10, PAD11, PAD12, PAD14, PAD20, PAD21, PAD23, PAD24: (no value), wirepad:SMD1.27-2.54
- added PAD3, PAD4, PAD5, PAD6, PAD7, PAD8: (no value), wirepad:SMD1.27-2.54
- moved PAD1 15.0 mm to (15.5, 15.0), flipped to the top, turned to 270 degrees
- moved PAD2 13.7 mm to (15.5, 15.0)
- moved R1 5.51 mm to (10.6, 21.4), turned to 180 degrees
Connections:
- removed net N$3: PAD14.1, R1.1
- new net N$2: PAD1.1, R1.1
- net N: now also PAD4.1, PAD6.1, PAD8.1; no longer PAD20.1, PAD21.1, PAD23.1, PAD24.1
- net S: now also PAD3.1, PAD5.1, PAD7.1; no longer PAD1.1, PAD10.1, PAD11.1, PAD12.1
Routing:
- net N$2: track 0.00 -> 8.55 mm
- net N$3: track 8.48 -> 0.00 mm
- net N: track 19.5 -> 23.5 mm
- added copper zone on layer 1, net N
- added copper zone on layer 1, net S
Other:
- board size 25.3 x 34.5 mm -> 25 x 29.5 mm
- board text added: "2012.01"
- board text removed: "2012.04"
- board text removed: "Add"
- board text removed: "DCC"
- board text removed: "here"
- board text removed: "weight"

Commit message: 1.1
Other:
- outline, holes or cut-outs redrawn
Changed lines of the file:
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@@
 <grid distance="50" unitdist="mil" unit="mil" style="dots" multiple="2" display="yes" altdistance="25" altunitdist="mil" altunit="mil"/>
 <layers>
-<layer number="1" name="Top" color="4" fill="1" visible="no" active="yes"/>
-<layer number="16" name="Bottom" color="2" fill="1" visible="no" active="yes"/>
+<layer number="1" name="Top" color="4" fill="1" visible="yes" active="yes"/>
+<layer number="16" name="Bottom" color="2" fill="1" visible="yes" active="yes"/>
 <layer number="17" name="Pads" color="23" fill="1" visible="yes" active="yes"/>
 <layer number="18" name="Vias" color="29" fill="1" visible="yes" active="yes"/>
-<layer number="19" name="Unrouted" color="6" fill="1" visible="no" active="yes"/>
+<layer number="19" name="Unrouted" color="6" fill="1" visible="yes" active="yes"/>
 <layer number="20" name="Dimension" color="15" fill="1" visible="yes" active="yes"/>
 <layer number="21" name="tPlace" color="19" fill="1" visible="yes" active="yes"/>
 <layer number="22" name="bPlace" color="17" fill="1" visible="no" active="yes"/>
-<layer number="23" name="tOrigins" color="30" fill="1" visible="no" active="yes"/>
+<layer number="23" name="tOrigins" color="30" fill="1" visible="yes" active="yes"/>
 <layer number="24" name="bOrigins" color="15" fill="1" visible="no" active="yes"/>
 <layer number="25" name="tNames" color="63" fill="1" visible="yes" active="yes"/>
@@
 <layer number="42" name="bRestrict" color="3" fill="10" visible="no" active="yes"/>
 <layer number="43" name="vRestrict" color="2" fill="10" visible="no" active="yes"/>
-<layer number="44" name="Drills" color="16" fill="1" visible="no" active="yes"/>
-<layer number="45" name="Holes" color="35" fill="1" visible="no" active="yes"/>
-<layer number="46" name="Milling" color="35" fill="1" visible="no" active="yes"/>
-<layer number="47" name="Measures" color="21" fill="1" visible="no" active="yes"/>
-<layer number="48" name="Document" color="24" fill="1" visible="no" active="yes"/>
-<layer number="49" name="Reference" color="48" fill="1" visible="no" active="yes"/>
+<layer number="44" name="Drills" color="16" fill="1" visible="yes" active="yes"/>
+<layer number="45" name="Holes" color="35" fill="1" visible="yes" active="yes"/>
+<layer number="46" name="Milling" color="35" fill="1" visible="yes" active="yes"/>
+<layer number="47" name="Measures" color="21" fill="1" visible="yes" active="yes"/>
+<layer number="48" name="Document" color="24" fill="1" visible="yes" active="yes"/>
+<layer number="49" name="Reference" color="48" fill="1" visible="yes" active="yes"/>
 <layer number="50" name="dxf" color="7" fill="1" visible="no" active="yes"/>
 <layer number="51" name="tDocu" color="24" fill="1" visible="yes" active="yes"/>
@@
 <wire x1="0" y1="0" x2="25" y2="0" width="0" layer="20"/>
 <wire x1="25" y1="0" x2="25" y2="13" width="0" layer="20"/>
-<wire x1="25" y1="13" x2="16" y2="13" width="0" layer="20"/>
-<wire x1="16" y1="13" x2="16" y2="14" width="0" layer="20"/>
-<wire x1="16" y1="14" x2="17" y2="14" width="0" layer="20"/>
-<wire x1="17" y1="14" x2="17" y2="16" width="0" layer="20"/>
-<wire x1="17" y1="16" x2="23" y2="20" width="0" layer="20"/>
-<wire x1="23" y1="20" x2="23" y2="24" width="0" layer="20"/>
-<wire x1="23" y1="24" x2="13" y2="28" width="0" layer="20"/>
-<wire x1="13" y1="28" x2="8" y2="29.5" width="0" layer="20"/>
-<wire x1="8" y1="29.5" x2="2" y2="26.5" width="0" layer="20"/>
-<wire x1="2" y1="26.5" x2="2" y2="16.5" width="0" layer="20"/>
-<wire x1="2" y1="16.5" x2="12.5" y2="14" width="0" layer="20"/>
+<wire x1="25" y1="13" x2="17" y2="13" width="0" layer="20"/>
 <wire x1="12.5" y1="13" x2="0" y2="13" width="0" layer="20"/>
 <wire x1="0" y1="13" x2="0" y2="0" width="0" layer="20"/>
-<wire x1="16" y1="24" x2="16" y2="19" width="0" layer="48" curve="-270"/>
-<wire x1="16" y1="19" x2="15" y2="20" width="0" layer="48"/>
-<wire x1="15" y1="20" x2="14" y2="19.5" width="0" layer="48"/>
-<wire x1="14" y1="19.5" x2="14" y2="16.5" width="0" layer="48"/>
-<wire x1="14" y1="16.5" x2="14.5" y2="16" width="0" layer="48"/>
-<wire x1="14.5" y1="16" x2="17" y2="16" width="0" layer="48"/>
-<wire x1="12.5" y1="14" x2="11.5" y2="15.5" width="0" layer="48"/>
-<wire x1="11.5" y1="15.5" x2="11.5" y2="18" width="0" layer="48"/>
-<wire x1="11.5" y1="18" x2="10" y2="19" width="0" layer="48"/>
-<wire x1="10" y1="19" x2="8" y2="18.5" width="0" layer="48"/>
-<wire x1="8" y1="18.5" x2="2" y2="16.5" width="0" layer="48"/>
-<wire x1="2" y1="16.5" x2="2" y2="20" width="0" layer="48"/>
-<wire x1="2" y1="20" x2="7" y2="20.5" width="0" layer="48"/>
-<wire x1="7" y1="20.5" x2="7" y2="22.5" width="0" layer="48"/>
-<wire x1="7" y1="22.5" x2="2" y2="23" width="0" layer="48"/>
-<wire x1="2" y1="23" x2="2" y2="26.5" width="0" layer="48"/>
-<wire x1="2" y1="26.5" x2="8.5" y2="24.5" width="0" layer="48"/>
-<wire x1="8.5" y1="24.5" x2="10.5" y2="24" width="0" layer="48"/>
-<wire x1="10.5" y1="24" x2="11.5" y2="25" width="0" layer="48"/>
-<wire x1="11.5" y1="25" x2="10.5" y2="26" width="0" layer="48"/>
-<wire x1="10.5" y1="26" x2="7" y2="28" width="0" layer="48"/>
-<wire x1="7" y1="28" x2="7" y2="29" width="0" layer="48"/>
-<wire x1="7" y1="29" x2="8" y2="29.5" width="0" layer="48"/>
-<wire x1="8" y1="29.5" x2="13" y2="28" width="0" layer="48"/>
-<wire x1="13" y1="28" x2="14" y2="27" width="0" layer="48"/>
-<wire x1="14" y1="27" x2="14" y2="23.5" width="0" layer="48"/>
-<wire x1="14" y1="23.5" x2="15.5" y2="23" width="0" layer="48"/>
-<wire x1="15.5" y1="23" x2="16" y2="24" width="0" layer="48"/>
+<wire x1="16" y1="24" x2="16" y2="19" width="0" layer="20" curve="-270"/>
+<wire x1="16" y1="19" x2="15" y2="20" width="0" layer="20"/>
+<wire x1="15" y1="20" x2="14" y2="19.5" width="0" layer="20"/>
+<wire x1="14" y1="19.5" x2="14" y2="16.5" width="0" layer="20"/>
+<wire x1="14" y1="16.5" x2="14.5" y2="16" width="0" layer="20"/>
+<wire x1="14.5" y1="16" x2="17" y2="16" width="0" layer="20"/>
+<wire x1="12.5" y1="14" x2="11.5" y2="15.5" width="0" layer="20"/>
+<wire x1="11.5" y1="15.5" x2="11.5" y2="18" width="0" layer="20"/>
+<wire x1="11.5" y1="18" x2="10" y2="19" width="0" layer="20"/>
+<wire x1="10" y1="19" x2="8" y2="18.5" width="0" layer="20"/>
+<wire x1="8" y1="18.5" x2="2" y2="16.5" width="0" layer="20"/>
+<wire x1="2" y1="16.5" x2="2" y2="20" width="0" layer="20"/>
+<wire x1="2" y1="20" x2="7" y2="20.5" width="0" layer="20"/>
+<wire x1="7" y1="20.5" x2="7" y2="22.5" width="0" layer="20"/>
+<wire x1="7" y1="22.5" x2="2" y2="23" width="0" layer="20"/>
+<wire x1="2" y1="23" x2="2" y2="26.5" width="0" layer="20"/>
+<wire x1="2" y1="26.5" x2="8.5" y2="24.5" width="0" layer="20"/>
+<wire x1="8.5" y1="24.5" x2="10.5" y2="24" width="0" layer="20"/>
+<wire x1="10.5" y1="24" x2="11.5" y2="25" width="0" layer="20"/>
+<wire x1="11.5" y1="25" x2="10.5" y2="26" width="0" layer="20"/>
+<wire x1="10.5" y1="26" x2="7" y2="28" width="0" layer="20"/>
+<wire x1="7" y1="28" x2="7" y2="29" width="0" layer="20"/>
+<wire x1="7" y1="29" x2="8" y2="29.5" width="0" layer="20"/>
+<wire x1="8" y1="29.5" x2="13" y2="28" width="0" layer="20"/>
+<wire x1="13" y1="28" x2="14" y2="27" width="0" layer="20"/>
+<wire x1="14" y1="27" x2="14" y2="23.5" width="0" layer="20"/>
+<wire x1="14" y1="23.5" x2="15.5" y2="23" width="0" layer="20"/>
+<wire x1="15.5" y1="23" x2="16" y2="24" width="0" layer="20"/>
 <wire x1="12.5" y1="14" x2="12.5" y2="13" width="0" layer="20"/>
-<wire x1="17" y1="16" x2="17" y2="14" width="0" layer="48"/>
-<wire x1="17" y1="14" x2="12.5" y2="14" width="0" layer="48"/>
-<wire x1="17.24" y1="23.32" x2="17.24" y2="19.51" width="0.254" layer="51" curve="119.997846"/>
-<wire x1="19" y1="22" x2="18" y2="21.5" width="0.254" layer="51"/>
-<wire x1="18" y1="21.5" x2="18" y2="22" width="0.254" layer="51"/>
+<wire x1="17" y1="16" x2="17" y2="13" width="0" layer="20"/>
+<wire x1="17.24" y1="23.32" x2="17.24" y2="19.51" width="0.254" layer="48" curve="119.997846"/>
+<wire x1="19" y1="22" x2="18" y2="21.5" width="0.254" layer="48"/>
+<wire x1="18" y1="21.5" x2="18" y2="22" width="0.254" layer="48"/>
 <wire x1="18" y1="23" x2="21.5" y2="23" width="0.254" layer="52"/>
 <wire x1="18" y1="21.5" x2="22" y2="21.5" width="0.254" layer="52"/>
@@
 <wire x1="18.5" y1="22" x2="22" y2="22" width="0.254" layer="52"/>
 <wire x1="18.5" y1="22.5" x2="22" y2="22.5" width="0.254" layer="52"/>
-<wire x1="50" y1="0" x2="50" y2="50" width="0.254" layer="19"/>
-<wire x1="50" y1="50" x2="0" y2="50" width="0.254" layer="19"/>
-<circle x="20" y="23" radius="0.5" width="0.254" layer="51"/>
-<circle x="20" y="20.5" radius="0.5" width="0.254" layer="51"/>
-<text x="12.5" y="25" size="1.016" layer="51" rot="SR270">Brakeman</text>
+<circle x="20" y="23" radius="0.5" width="0.254" layer="48"/>
+<circle x="20" y="20.5" radius="0.5" width="0.254" layer="48"/>
+<text x="12.5" y="25" size="1.016" layer="48" rot="SR270">Brakeman</text>
 <text x="12.5" y="19" size="1.016" layer="52" rot="SMR90">Safety</text>
 <text x="10.5" y="19.5" size="1.016" layer="52" rot="SMR90">First!</text>

Commit message: 1.2
Parts:
- removed PAD3, PAD4, PAD5, PAD6, PAD7, PAD8: (no value), wirepad:SMD1.27-2.54
- added PAD10, PAD11, PAD12, PAD14, PAD20, PAD21, PAD23, PAD24: (no value), wirepad:SMD1.27-2.54
- moved PAD1 15.0 mm to (9.53, 1.27), flipped to the bottom, turned to 90 degrees
- moved PAD2 13.7 mm to (15.9, 1.27)
- moved R1 5.51 mm to (9.02, 26.7), turned to 90 degrees
Connections:
- removed net N$2: PAD1.1, R1.1
- new net N$3: PAD14.1, R1.1
- net N: now also PAD20.1, PAD21.1, PAD23.1, PAD24.1; no longer PAD4.1, PAD6.1, PAD8.1
- net S: now also PAD1.1, PAD10.1, PAD11.1, PAD12.1; no longer PAD3.1, PAD5.1, PAD7.1
Routing:
- net N$2: track 8.55 -> 0.00 mm
- net N$3: track 0.00 -> 8.48 mm
- net N: track 23.5 -> 19.5 mm
- removed copper zone on layer 1, net N
- removed copper zone on layer 1, net S
Other:
- board size 25 x 29.5 mm -> 25.3 x 34.5 mm
- board text added: "2012.04"
- board text added: "Add"
- board text added: "DCC"
- board text added: "here"
- board text added: "weight"
- board text removed: "2012.01"

Commit message: 1.3
Parts:
- removed PAD1, PAD10, PAD11, PAD12, PAD14, PAD2, PAD20, PAD21, PAD23, PAD24: (no value), wirepad:SMD1.27-2.54
- added PADL1, PADL2, PADN2, PADN3, PADN4, PADN6, PADS2, PADS4: (no value), wirepad:SMD1.27-2.54
- R1: value (none) -> 1k0; device resistor:R0805 -> resistor:0204/5
- moved R1 1.42 mm to (10.3, 27.3), flipped to the bottom
Connections:
- removed net N$3: PAD14.1, R1.1
- new net LIMITED: PADL1.1, PADL2.1, R1.1
- net N: now also PADN2.1, PADN3.1, PADN4.1, PADN6.1; no longer PAD2.1, PAD20.1, PAD21.1, PAD23.1, PAD24.1
- net S: now also PADS2.1, PADS4.1; no longer PAD1.1, PAD10.1, PAD11.1, PAD12.1
Routing:
- net LIMITED: track 0.00 -> 19.7 mm
- net N: track 19.5 -> 31.5 mm
- net N$3: track 8.48 -> 0.00 mm
- net S: track 11.0 -> 12.0 mm
Other:
- board size 25.3 x 34.5 mm -> 22.6 x 34.5 mm
- board text added: "2016.04"
- board text added: "DCC Flagman & Fusee"
- board text added: "Flagman"
- board text added: "www.SPCoast.com"
- board text removed: "2012.04"
- board text removed: "Brakeman"
- board text removed: "DCC Brakeman"

Commit message: 2.0
Parts:
- removed PADN2, PADN3, PADN4, PADN6, PADS2, PADS4: (no value), wirepad:SMD1.27-2.54
- added PADNA, PADNA2, PADNF, PADNF2, PADSF, PADSF2: (no value), wirepad:SMD1.27-2.54
- moved PADL2 10.9 mm to (18.3, 33.7), turned to 0 degrees
- moved PADL1 10.8 mm to (5.05, 26.2), turned to 160 degrees
- moved R1 3.02 mm to (11.9, 29.8), turned to 0 degrees
Connections:
- net N: now also PADNA.1, PADNA2.1, PADNF.1, PADNF2.1; no longer PADN2.1, PADN3.1, PADN4.1, PADN6.1
- net S: now also PADSF.1, PADSF2.1; no longer PADS2.1, PADS4.1
Routing:
- net S: track 12.0 -> 19.7 mm
- net N: track 31.5 -> 38.9 mm
- added copper zone on layer 1, net N
- added copper zone on layer 1, net S
Other:
- board size 22.6 x 34.5 mm -> 23.9 x 39.6 mm
- board text added: "DCC Flagman"
- board text removed: "DCC Flagman & Fusee"

Commit message: 2.1
Parts:
- moved PADL1 27.2 mm to (16.8, 1.65), turned to 250 degrees
- moved PADNA 27.2 mm to (16.8, 1.65), turned to 110 degrees
- moved R1 21.4 mm to (13.1, 8.51), turned to 270 degrees
- moved PADL2 20.8 mm to (9.27, 14.9), turned to 90 degrees
- moved PADNA2 20.8 mm to (9.27, 14.9), turned to 270 degrees
- moved PADSF 20.6 mm to (23.2, 5.31), turned to 180 degrees
- moved PADSF2 20.6 mm to (23.2, 5.31), turned to 180 degrees
- moved PADNF 11.9 mm to (23.2, 11.5), turned to 180 degrees
- moved PADNF2 11.9 mm to (23.2, 11.5), turned to 180 degrees
Routing:
- net S: track 19.7 -> 51.5 mm
- net N: track 38.9 -> 62.7 mm, vias 2 -> 3
Other:
- board size 23.9 x 39.6 mm -> 25.4 x 37.7 mm
- board text added: "V-Score"

Commit message: 2.2
Parts:
- moved PADNF 51.8 mm to (23.0, 63.3)
- moved PADL1 51.8 mm to (16.5, 53.5)
- moved PADL2 51.8 mm to (9.04, 66.7)
- moved PADNA 51.8 mm to (16.5, 53.5)
- moved PADNA2 51.8 mm to (9.04, 66.7)
- moved PADNF2 51.8 mm to (23.0, 63.3)
- moved PADSF 51.8 mm to (23.0, 57.1)
- moved PADSF2 51.8 mm to (23.0, 57.1)
- moved R1 51.8 mm to (12.9, 60.3)
Other:
- board size 25.4 x 37.7 mm -> 23.6 x 43.2 mm
- board text removed: "V-Score"

Commit message: 2.3
Parts:
- moved PADNF2 44.1 mm to (14.9, 20.0), flipped to the top, turned to 90 degrees
- moved PADNF 44.1 mm to (14.9, 20.0), flipped to the bottom, turned to 270 degrees
- moved PADL2 40.6 mm to (5.82, 26.2), turned to 160 degrees
- moved PADNA2 40.6 mm to (5.82, 26.2), turned to 200 degrees
- moved PADSF 39.8 mm to (8.71, 20.0), flipped to the bottom, turned to 270 degrees
- moved PADSF2 39.8 mm to (8.71, 20.0), flipped to the top, turned to 90 degrees
- moved R1 30.5 mm to (11.9, 29.8), turned to 0 degrees
- moved PADL1 19.9 mm to (18.3, 33.7), turned to 0 degrees
- moved PADNA 19.9 mm to (18.3, 33.7), turned to 0 degrees
Routing:
- net S: track 51.5 -> 19.7 mm
- net N: track 62.7 -> 38.6 mm, vias 3 -> 2
Other:
- board size 23.6 x 43.2 mm -> 37.3 x 48.3 mm
- board text added: "2016.11"
- board text added: "Safety Sam"
- board text added: "V-Groove"
- board text removed: "2016.04"
