File: Brakeman.sch (EAGLE design)
At the start: 11 parts

Commit message: 1.0
Parts:
- removed PAD10, PAD11, PAD12, PAD14, PAD20, PAD21, PAD23, PAD24: (no value), wirepad:SMD2
- added PAD3, PAD4, PAD5, PAD6, PAD7, PAD8: (no value), wirepad:SMD2
Connections:
- removed net N$3: PAD14.P, R1.1
- new net N$2: PAD1.P, R1.1
- net N: now also PAD4.P, PAD6.P, PAD8.P; no longer PAD20.P, PAD21.P, PAD23.P, PAD24.P
- net S: now also PAD3.P, PAD5.P, PAD7.P; no longer PAD1.P, PAD10.P, PAD11.P, PAD12.P
Other:
- note added: "DCC Flangman/Brakeman"
- note added: "v1.0"
- note removed: "DCC Flagman/Brakeman"
- note removed: "V0.0"
- moved on the sheet: PAD1, PAD2, R1
Changed lines of the file:
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@@
 <part name="FRAME1" library="SparkFun" deviceset="FRAME-LETTER" device=""/>
 <part name="R1" library="resistor" deviceset="R-US_" device="R0805"/>
-<part name="PAD23" library="wirepad" deviceset="SMD2" device=""/>
-<part name="PAD10" library="wirepad" deviceset="SMD2" device=""/>
-<part name="PAD20" library="wirepad" deviceset="SMD2" device=""/>
-<part name="PAD11" library="wirepad" deviceset="SMD2" device=""/>
-<part name="PAD21" library="wirepad" deviceset="SMD2" device=""/>
-<part name="PAD12" library="wirepad" deviceset="SMD2" device=""/>
-<part name="PAD14" library="wirepad" deviceset="SMD2" device=""/>
-<part name="PAD24" library="wirepad" deviceset="SMD2" device=""/>
 <part name="PAD1" library="wirepad" deviceset="SMD2" device=""/>
 <part name="PAD2" library="wirepad" deviceset="SMD2" device=""/>
+<part name="PAD3" library="wirepad" deviceset="SMD2" device=""/>
+<part name="PAD4" library="wirepad" deviceset="SMD2" device=""/>
+<part name="PAD5" library="wirepad" deviceset="SMD2" device=""/>
+<part name="PAD6" library="wirepad" deviceset="SMD2" device=""/>
+<part name="PAD7" library="wirepad" deviceset="SMD2" device=""/>
+<part name="PAD8" library="wirepad" deviceset="SMD2" device=""/>
 </parts>
 <sheets>
 <sheet>
 <plain>
-<text x="238.76" y="7.62" size="1.778" layer="91">V0.0</text>
-<text x="152.4" y="27.94" size="2.54" layer="91">DCC Flagman/Brakeman</text>
+<text x="152.4" y="27.94" size="2.54" layer="91">DCC Flangman/Brakeman</text>
+<text x="236.22" y="7.62" size="2.54" layer="91">v1.0</text>
 </plain>
 <instances>
 <instance part="FRAME1" gate="G$1" x="0" y="0"/>
 <instance part="FRAME1" gate="G$2" x="147.32" y="0"/>
-<instance part="R1" gate="G$1" x="104.14" y="96.52" rot="R270"/>
-<instance part="PAD23" gate="1" x="81.28" y="91.44"/>
-<instance part="PAD10" gate="1" x="106.68" y="76.2" rot="R180"/>
-<instance part="PAD20" gate="1" x="81.28" y="76.2"/>
-<instance part="PAD11" gate="1" x="106.68" y="81.28" rot="R180"/>
-<instance part="PAD21" gate="1" x="81.28" y="81.28"/>
-<instance part="PAD12" gate="1" x="106.68" y="88.9" rot="R180"/>
-<instance part="PAD14" gate="1" x="106.68" y="104.14" rot="R180"/>
-<instance part="PAD24" gate="1" x="81.28" y="96.52"/>
-<instance part="PAD1" gate="1" x="106.68" y="83.82" rot="R180"/>
-<instance part="PAD2" gate="1" x="81.28" y="101.6"/>
+<instance part="R1" gate="G$1" x="43.18" y="160.02" rot="R90"/>
+<instance part="PAD1" gate="1" x="40.64" y="154.94"/>
+<instance part="PAD2" gate="1" x="40.64" y="147.32"/>
+<instance part="PAD3" gate="1" x="40.64" y="167.64"/>
+<instance part="PAD4" gate="1" x="40.64" y="142.24"/>
+<instance part="PAD5" gate="1" x="40.64" y="165.1"/>
+<instance part="PAD6" gate="1" x="40.64" y="144.78"/>
+<instance part="PAD7" gate="1" x="45.72" y="165.1" rot="R180"/>
+<instance part="PAD8" gate="1" x="45.72" y="147.32" rot="R180"/>
 </instances>
 <busses>
 </busses>
 <nets>
+<net name="N$2" class="0">
+<segment>
+<pinref part="R1" gate="G$1" pin="1"/>
+<pinref part="PAD1" gate="1" pin="P"/>
+</segment>
+</net>
 <net name="N" class="0">
 <segment>
-<wire x1="83.82" y1="81.28" x2="83.82" y2="76.2" width="0.1524" layer="91"/>
-<junction x="83.82" y="81.28"/>
-<label x="83.82" y="76.2" size="1.778" layer="95" xref="yes"/>
-<pinref part="PAD23" gate="1" pin="P"/>
-<pinref part="PAD20" gate="1" pin="P"/>
-<pinref part="PAD21" gate="1" pin="P"/>
-<wire x1="83.82" y1="81.28" x2="83.82" y2="91.44" width="0.1524" layer="91"/>
-<pinref part="PAD24" gate="1" pin="P"/>
-<wire x1="83.82" y1="91.44" x2="83.82" y2="96.52" width="0.1524" layer="91"/>
-<junction x="83.82" y="91.44"/>
+<wire x1="43.18" y1="147.32" x2="43.18" y2="144.78" width="0.1524" layer="91"/>
+<wire x1="43.18" y1="144.78" x2="43.18" y2="142.24" width="0.1524" layer="91"/>
+<junction x="43.18" y="144.78"/>
+<junction x="43.18" y="147.32"/>
+<label x="43.18" y="142.24" size="1.778" layer="95" xref="yes"/>
 <pinref part="PAD2" gate="1" pin="P"/>
-<wire x1="83.82" y1="96.52" x2="83.82" y2="101.6" width="0.1524" layer="91"/>
-<junction x="83.82" y="96.52"/>
+<pinref part="PAD4" gate="1" pin="P"/>
+<pinref part="PAD6" gate="1" pin="P"/>
+<pinref part="PAD8" gate="1" pin="P"/>
 </segment>
 </net>
 <net name="S" class="0">
 <segment>
-<wire x1="104.14" y1="91.44" x2="104.14" y2="88.9" width="0.1524" layer="91"/>
-<label x="104.14" y="76.2" size="1.778" layer="95" rot="R180" xref="yes"/>
+<wire x1="43.18" y1="165.1" x2="43.18" y2="167.64" width="0.1524" layer="91"/>
+<junction x="43.18" y="165.1"/>
+<label x="43.18" y="167.64" size="1.778" layer="95" xref="yes"/>
 <pinref part="R1" gate="G$1" pin="2"/>
-<pinref part="PAD10" gate="1" pin="P"/>
-<pinref part="PAD12" gate="1" pin="P"/>
-<junction x="104.14" y="88.9"/>
-<wire x1="104.14" y1="88.9" x2="104.14" y2="83.82" width="0.1524" layer="91"/>
-<pinref part="PAD11" gate="1" pin="P"/>
-<junction x="104.14" y="81.28"/>
-<wire x1="104.14" y1="83.82" x2="104.14" y2="81.28" width="0.1524" layer="91"/>
-<wire x1="104.14" y1="81.28" x2="104.14" y2="76.2" width="0.1524" layer="91"/>
-<pinref part="PAD1" gate="1" pin="P"/>
-<junction x="104.14" y="83.82"/>
+<pinref part="PAD3" gate="1" pin="P"/>
+<pinref part="PAD5" gate="1" pin="P"/>
+<pinref part="PAD7" gate="1" pin="P"/>
 </segment>
 </net>
-<net name="N$3" class="0">
-<segment>
-<pinref part="R1" gate="G$1" pin="1"/>
-<wire x1="104.14" y1="101.6" x2="104.14" y2="104.14" width="0.1524" layer="91"/>
-<pinref part="PAD14" gate="1" pin="P"/>
-</segment>
-</net>

Commit message: 1.1
Other:
- note added: "DCC Flagman/Brakeman"
- note added: "V1.1"
- note removed: "DCC Flangman/Brakeman"
- note removed: "v1.0"
Changed lines of the file:
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@@
 <sheet>
 <plain>
-<text x="152.4" y="27.94" size="2.54" layer="91">DCC Flangman/Brakeman</text>
-<text x="236.22" y="7.62" size="2.54" layer="91">v1.0</text>
+<text x="154.94" y="27.94" size="2.54" layer="91">DCC Flagman/Brakeman</text>
+<text x="238.76" y="7.62" size="2.54" layer="91">V1.1</text>
 </plain>
 <instances>

Commit message: 1.2
Parts:
- removed PAD3, PAD4, PAD5, PAD6, PAD7, PAD8: (no value), wirepad:SMD2
- added PAD10, PAD11, PAD12, PAD14, PAD20, PAD21, PAD23, PAD24: (no value), wirepad:SMD2
Connections:
- removed net N$2: PAD1.P, R1.1
- new net N$3: PAD14.P, R1.1
- net N: now also PAD20.P, PAD21.P, PAD23.P, PAD24.P; no longer PAD4.P, PAD6.P, PAD8.P
- net S: now also PAD1.P, PAD10.P, PAD11.P, PAD12.P; no longer PAD3.P, PAD5.P, PAD7.P
Other:
- note added: "V1.2"
- note removed: "V1.1"
- moved on the sheet: PAD1, PAD2, R1
Changed lines of the file:
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@@
 <part name="FRAME1" library="SparkFun" deviceset="FRAME-LETTER" device=""/>
 <part name="R1" library="resistor" deviceset="R-US_" device="R0805"/>
+<part name="PAD23" library="wirepad" deviceset="SMD2" device=""/>
+<part name="PAD10" library="wirepad" deviceset="SMD2" device=""/>
+<part name="PAD20" library="wirepad" deviceset="SMD2" device=""/>
+<part name="PAD11" library="wirepad" deviceset="SMD2" device=""/>
+<part name="PAD21" library="wirepad" deviceset="SMD2" device=""/>
+<part name="PAD12" library="wirepad" deviceset="SMD2" device=""/>
+<part name="PAD14" library="wirepad" deviceset="SMD2" device=""/>
+<part name="PAD24" library="wirepad" deviceset="SMD2" device=""/>
 <part name="PAD1" library="wirepad" deviceset="SMD2" device=""/>
 <part name="PAD2" library="wirepad" deviceset="SMD2" device=""/>
-<part name="PAD3" library="wirepad" deviceset="SMD2" device=""/>
-<part name="PAD4" library="wirepad" deviceset="SMD2" device=""/>
-<part name="PAD5" library="wirepad" deviceset="SMD2" device=""/>
-<part name="PAD6" library="wirepad" deviceset="SMD2" device=""/>
-<part name="PAD7" library="wirepad" deviceset="SMD2" device=""/>
-<part name="PAD8" library="wirepad" deviceset="SMD2" device=""/>
 </parts>
 <sheets>
 <sheet>
 <plain>
-<text x="154.94" y="27.94" size="2.54" layer="91">DCC Flagman/Brakeman</text>
-<text x="238.76" y="7.62" size="2.54" layer="91">V1.1</text>
+<text x="236.22" y="7.62" size="2.54" layer="91">V1.2</text>
+<text x="149.86" y="27.94" size="2.54" layer="91">DCC Flagman/Brakeman</text>
 </plain>
 <instances>
 <instance part="FRAME1" gate="G$1" x="0" y="0"/>
 <instance part="FRAME1" gate="G$2" x="147.32" y="0"/>
-<instance part="R1" gate="G$1" x="43.18" y="160.02" rot="R90"/>
-<instance part="PAD1" gate="1" x="40.64" y="154.94"/>
-<instance part="PAD2" gate="1" x="40.64" y="147.32"/>
-<instance part="PAD3" gate="1" x="40.64" y="167.64"/>
-<instance part="PAD4" gate="1" x="40.64" y="142.24"/>
-<instance part="PAD5" gate="1" x="40.64" y="165.1"/>
-<instance part="PAD6" gate="1" x="40.64" y="144.78"/>
-<instance part="PAD7" gate="1" x="45.72" y="165.1" rot="R180"/>
-<instance part="PAD8" gate="1" x="45.72" y="147.32" rot="R180"/>
+<instance part="R1" gate="G$1" x="104.14" y="96.52" rot="R270"/>
+<instance part="PAD23" gate="1" x="81.28" y="91.44"/>
+<instance part="PAD10" gate="1" x="106.68" y="76.2" rot="R180"/>
+<instance part="PAD20" gate="1" x="81.28" y="76.2"/>
+<instance part="PAD11" gate="1" x="106.68" y="81.28" rot="R180"/>
+<instance part="PAD21" gate="1" x="81.28" y="81.28"/>
+<instance part="PAD12" gate="1" x="106.68" y="88.9" rot="R180"/>
+<instance part="PAD14" gate="1" x="106.68" y="104.14" rot="R180"/>
+<instance part="PAD24" gate="1" x="81.28" y="96.52"/>
+<instance part="PAD1" gate="1" x="106.68" y="83.82" rot="R180"/>
+<instance part="PAD2" gate="1" x="81.28" y="101.6"/>
 </instances>
 <busses>
 </busses>
 <nets>
-<net name="N$2" class="0">
-<segment>
-<pinref part="R1" gate="G$1" pin="1"/>
-<pinref part="PAD1" gate="1" pin="P"/>
-</segment>
-</net>
 <net name="N" class="0">
 <segment>
-<wire x1="43.18" y1="147.32" x2="43.18" y2="144.78" width="0.1524" layer="91"/>
-<wire x1="43.18" y1="144.78" x2="43.18" y2="142.24" width="0.1524" layer="91"/>
-<junction x="43.18" y="144.78"/>
-<junction x="43.18" y="147.32"/>
-<label x="43.18" y="142.24" size="1.778" layer="95" xref="yes"/>
+<wire x1="83.82" y1="81.28" x2="83.82" y2="76.2" width="0.1524" layer="91"/>
+<junction x="83.82" y="81.28"/>
+<label x="83.82" y="76.2" size="1.778" layer="95" xref="yes"/>
+<pinref part="PAD23" gate="1" pin="P"/>
+<pinref part="PAD20" gate="1" pin="P"/>
+<pinref part="PAD21" gate="1" pin="P"/>
+<wire x1="83.82" y1="81.28" x2="83.82" y2="91.44" width="0.1524" layer="91"/>
+<pinref part="PAD24" gate="1" pin="P"/>
+<wire x1="83.82" y1="91.44" x2="83.82" y2="96.52" width="0.1524" layer="91"/>
+<junction x="83.82" y="91.44"/>
 <pinref part="PAD2" gate="1" pin="P"/>
-<pinref part="PAD4" gate="1" pin="P"/>
-<pinref part="PAD6" gate="1" pin="P"/>
-<pinref part="PAD8" gate="1" pin="P"/>
+<wire x1="83.82" y1="96.52" x2="83.82" y2="101.6" width="0.1524" layer="91"/>
+<junction x="83.82" y="96.52"/>
 </segment>
 </net>
 <net name="S" class="0">
 <segment>
-<wire x1="43.18" y1="165.1" x2="43.18" y2="167.64" width="0.1524" layer="91"/>
-<junction x="43.18" y="165.1"/>
-<label x="43.18" y="167.64" size="1.778" layer="95" xref="yes"/>
+<wire x1="104.14" y1="91.44" x2="104.14" y2="88.9" width="0.1524" layer="91"/>
+<label x="104.14" y="76.2" size="1.778" layer="95" rot="R180" xref="yes"/>
 <pinref part="R1" gate="G$1" pin="2"/>
-<pinref part="PAD3" gate="1" pin="P"/>
-<pinref part="PAD5" gate="1" pin="P"/>
-<pinref part="PAD7" gate="1" pin="P"/>
+<pinref part="PAD10" gate="1" pin="P"/>
+<pinref part="PAD12" gate="1" pin="P"/>
+<junction x="104.14" y="88.9"/>
+<wire x1="104.14" y1="88.9" x2="104.14" y2="83.82" width="0.1524" layer="91"/>
+<pinref part="PAD11" gate="1" pin="P"/>
+<junction x="104.14" y="81.28"/>
+<wire x1="104.14" y1="83.82" x2="104.14" y2="81.28" width="0.1524" layer="91"/>
+<wire x1="104.14" y1="81.28" x2="104.14" y2="76.2" width="0.1524" layer="91"/>
+<pinref part="PAD1" gate="1" pin="P"/>
+<junction x="104.14" y="83.82"/>
 </segment>
 </net>
+<net name="N$3" class="0">
+<segment>
+<pinref part="R1" gate="G$1" pin="1"/>
+<wire x1="104.14" y1="101.6" x2="104.14" y2="104.14" width="0.1524" layer="91"/>
+<pinref part="PAD14" gate="1" pin="P"/>
+</segment>
+</net>

Commit message: 1.3
Parts:
- removed PAD1, PAD10, PAD11, PAD12, PAD14, PAD2, PAD20, PAD21, PAD23, PAD24: (no value), wirepad:SMD2
- added PADL1, PADL2, PADN2, PADN3, PADN4, PADN6, PADS2, PADS4: (no value), wirepad:SMD2
- R1: value (none) -> 1k0; device resistor:R-US_R0805 -> resistor:R-US_0204/5
Connections:
- removed net N$3: PAD14.P, R1.1
- new net LIMITED: PADL1.P, PADL2.P, R1.1
- net N: now also PADN2.P, PADN3.P, PADN4.P, PADN6.P; no longer PAD2.P, PAD20.P, PAD21.P, PAD23.P, PAD24.P
- net S: now also PADS2.P, PADS4.P; no longer PAD1.P, PAD10.P, PAD11.P, PAD12.P
Other:
- note added: "V1.3"
- note removed: "V1.2"
- moved on the sheet: R1

Commit message: 2.0
Parts:
- removed PADN2, PADN3, PADN4, PADN6, PADS2, PADS4: (no value), wirepad:SMD2
- added PADNA, PADNA2, PADNF, PADNF2, PADSF, PADSF2: (no value), wirepad:SMD2
Connections:
- net N: now also PADNA.P, PADNA2.P, PADNF.P, PADNF2.P; no longer PADN2.P, PADN3.P, PADN4.P, PADN6.P
- net S: now also PADSF.P, PADSF2.P; no longer PADS2.P, PADS4.P
Other:
- note added: "N"
- note added: "V2.0"
- note removed: "V1.3"
- moved on the sheet: PADL1, PADL2, R1
Changed lines of the file:
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@@
 <part name="FRAME1" library="SparkFun" deviceset="FRAME-LETTER" device=""/>
 <part name="R1" library="resistor" deviceset="R-US_" device="0204/5" value="1k0"/>
-<part name="PADN3" library="wirepad" deviceset="SMD2" device=""/>
-<part name="PADS2" library="wirepad" deviceset="SMD2" device=""/>
-<part name="PADN2" library="wirepad" deviceset="SMD2" device=""/>
-<part name="PADS4" library="wirepad" deviceset="SMD2" device=""/>
+<part name="PADNF2" library="wirepad" deviceset="SMD2" device=""/>
+<part name="PADSF" library="wirepad" deviceset="SMD2" device=""/>
+<part name="PADNF" library="wirepad" deviceset="SMD2" device=""/>
+<part name="PADSF2" library="wirepad" deviceset="SMD2" device=""/>
 <part name="PADL1" library="wirepad" deviceset="SMD2" device=""/>
-<part name="PADN4" library="wirepad" deviceset="SMD2" device=""/>
-<part name="PADN6" library="wirepad" deviceset="SMD2" device=""/>
+<part name="PADNA" library="wirepad" deviceset="SMD2" device=""/>
+<part name="PADNA2" library="wirepad" deviceset="SMD2" device=""/>
 <part name="PADL2" library="wirepad" deviceset="SMD2" device=""/>
 </parts>
@@
 <sheet>
 <plain>
+<text x="66.04" y="78.74" size="1.27" layer="91">N</text>
+<text x="238.76" y="7.62" size="2.54" layer="91">V2.0</text>
 <text x="154.94" y="27.94" size="2.54" layer="91">DCC Flagman/Brakeman</text>
-<text x="236.22" y="7.62" size="2.54" layer="91">V1.3</text>
 </plain>
 <instances>
 <instance part="FRAME1" gate="G$1" x="0" y="0"/>
 <instance part="FRAME1" gate="G$2" x="147.32" y="0"/>
-<instance part="R1" gate="G$1" x="40.64" y="137.16" rot="R270"/>
-<instance part="PADN3" gate="1" x="17.78" y="124.46"/>
-<instance part="PADS2" gate="1" x="43.18" y="114.3" rot="R180"/>
-<instance part="PADN2" gate="1" x="17.78" y="114.3"/>
-<instance part="PADS4" gate="1" x="43.18" y="129.54" rot="R180"/>
-<instance part="PADL1" gate="1" x="43.18" y="144.78" rot="R180"/>
-<instance part="PADN4" gate="1" x="17.78" y="129.54"/>
-<instance part="PADN6" gate="1" x="17.78" y="139.7"/>
-<instance part="PADL2" gate="1" x="43.18" y="149.86" rot="R180"/>
+<instance part="R1" gate="G$1" x="88.9" y="106.68" rot="R270"/>
+<instance part="PADNF2" gate="1" x="66.04" y="93.98"/>
+<instance part="PADSF" gate="1" x="91.44" y="86.36" rot="R180"/>
+<instance part="PADNF" gate="1" x="66.04" y="86.36"/>
+<instance part="PADSF2" gate="1" x="91.44" y="93.98" rot="R180"/>
+<instance part="PADL1" gate="1" x="91.44" y="124.46" rot="R180"/>
+<instance part="PADNA" gate="1" x="66.04" y="104.14"/>
+<instance part="PADNA2" gate="1" x="66.04" y="111.76"/>
+<instance part="PADL2" gate="1" x="91.44" y="132.08" rot="R180"/>
 </instances>
 <busses>
@@
 <net name="N" class="0">
 <segment>
-<wire x1="20.32" y1="114.3" x2="20.32" y2="109.22" width="0.1524" layer="91"/>
-<junction x="20.32" y="114.3"/>
-<label x="20.32" y="109.22" size="1.778" layer="95" xref="yes"/>
-<pinref part="PADN3" gate="1" pin="P"/>
-<pinref part="PADN2" gate="1" pin="P"/>
-<wire x1="20.32" y1="114.3" x2="20.32" y2="124.46" width="0.1524" layer="91"/>
-<pinref part="PADN4" gate="1" pin="P"/>
-<wire x1="20.32" y1="124.46" x2="20.32" y2="129.54" width="0.1524" layer="91"/>
-<junction x="20.32" y="124.46"/>
-<junction x="20.32" y="129.54"/>
-<pinref part="PADN6" gate="1" pin="P"/>
-<wire x1="20.32" y1="129.54" x2="20.32" y2="139.7" width="0.1524" layer="91"/>
+<pinref part="PADNF" gate="1" pin="P"/>
+<wire x1="68.58" y1="86.36" x2="76.2" y2="86.36" width="0.1524" layer="91"/>
+<wire x1="76.2" y1="86.36" x2="76.2" y2="93.98" width="0.1524" layer="91"/>
+<pinref part="PADNA2" gate="1" pin="P"/>
+<wire x1="76.2" y1="93.98" x2="76.2" y2="104.14" width="0.1524" layer="91"/>
+<wire x1="76.2" y1="104.14" x2="76.2" y2="111.76" width="0.1524" layer="91"/>
+<wire x1="76.2" y1="111.76" x2="68.58" y2="111.76" width="0.1524" layer="91"/>
+<pinref part="PADNA" gate="1" pin="P"/>
+<wire x1="68.58" y1="104.14" x2="76.2" y2="104.14" width="0.1524" layer="91"/>
+<junction x="76.2" y="104.14"/>
+<pinref part="PADNF2" gate="1" pin="P"/>
+<wire x1="68.58" y1="93.98" x2="76.2" y2="93.98" width="0.1524" layer="91"/>
+<junction x="76.2" y="93.98"/>
 </segment>
 </net>
 <net name="S" class="0">
 <segment>
-<wire x1="40.64" y1="132.08" x2="40.64" y2="129.54" width="0.1524" layer="91"/>
-<label x="40.64" y="109.22" size="1.778" layer="95" rot="R180" xref="yes"/>
+<pinref part="PADSF" gate="1" pin="P"/>
+<wire x1="88.9" y1="86.36" x2="83.82" y2="86.36" width="0.1524" layer="91"/>
+<wire x1="83.82" y1="86.36" x2="83.82" y2="93.98" width="0.1524" layer="91"/>
+<pinref part="PADSF2" gate="1" pin="P"/>
+<wire x1="83.82" y1="93.98" x2="88.9" y2="93.98" width="0.1524" layer="91"/>
 <pinref part="R1" gate="G$1" pin="2"/>
-<pinref part="PADS4" gate="1" pin="P"/>
-<junction x="40.64" y="129.54"/>
-<pinref part="PADS2" gate="1" pin="P"/>
-<junction x="40.64" y="114.3"/>
-<wire x1="40.64" y1="129.54" x2="40.64" y2="114.3" width="0.1524" layer="91"/>
-<wire x1="40.64" y1="114.3" x2="40.64" y2="109.22" width="0.1524" layer="91"/>
+<wire x1="88.9" y1="101.6" x2="83.82" y2="101.6" width="0.1524" layer="91"/>
+<wire x1="83.82" y1="101.6" x2="83.82" y2="93.98" width="0.1524" layer="91"/>
+<junction x="83.82" y="93.98"/>
 </segment>
 </net>
@@
 <segment>
 <pinref part="R1" gate="G$1" pin="1"/>
-<wire x1="40.64" y1="142.24" x2="40.64" y2="144.78" width="0.1524" layer="91"/>
+<wire x1="88.9" y1="111.76" x2="83.82" y2="111.76" width="0.1524" layer="91"/>
+<wire x1="83.82" y1="111.76" x2="83.82" y2="124.46" width="0.1524" layer="91"/>
 <pinref part="PADL1" gate="1" pin="P"/>
+<wire x1="83.82" y1="124.46" x2="88.9" y2="124.46" width="0.1524" layer="91"/>
 <pinref part="PADL2" gate="1" pin="P"/>
-<wire x1="40.64" y1="144.78" x2="40.64" y2="149.86" width="0.1524" layer="91"/>
-<junction x="40.64" y="144.78"/>
+<wire x1="88.9" y1="132.08" x2="83.82" y2="132.08" width="0.1524" layer="91"/>
+<wire x1="83.82" y1="132.08" x2="83.82" y2="124.46" width="0.1524" layer="91"/>
+<junction x="83.82" y="124.46"/>
 </segment>
 </net>

Commit message: 2.1
Other:
- note added: "V2.1"
- note removed: "V2.0"
Changed lines of the file:
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@@
 <plain>
 <text x="66.04" y="78.74" size="1.27" layer="91">N</text>
-<text x="238.76" y="7.62" size="2.54" layer="91">V2.0</text>
-<text x="154.94" y="27.94" size="2.54" layer="91">DCC Flagman/Brakeman</text>
+<text x="149.86" y="27.94" size="2.54" layer="91">DCC Flagman/Brakeman</text>
+<text x="238.76" y="7.62" size="2.54" layer="91">V2.1</text>
 </plain>
 <instances>

Commit message: 2.2
Other:
- note added: "V2.2"
- note removed: "V2.1"
Changed lines of the file:
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@@
 <plain>
 <text x="66.04" y="78.74" size="1.27" layer="91">N</text>
-<text x="149.86" y="27.94" size="2.54" layer="91">DCC Flagman/Brakeman</text>
-<text x="238.76" y="7.62" size="2.54" layer="91">V2.1</text>
+<text x="236.22" y="7.62" size="2.54" layer="91">V2.2</text>
+<text x="152.4" y="27.94" size="2.54" layer="91">DCC Flagman/Brakeman</text>
 </plain>
 <instances>

Commit message: 2.3
Other:
- note added: "V2.3"
- note removed: "V2.2"
Changed lines of the file:
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@@
 <plain>
 <text x="66.04" y="78.74" size="1.27" layer="91">N</text>
-<text x="236.22" y="7.62" size="2.54" layer="91">V2.2</text>
-<text x="152.4" y="27.94" size="2.54" layer="91">DCC Flagman/Brakeman</text>
+<text x="154.94" y="27.94" size="2.54" layer="91">DCC Flagman/Brakeman</text>
+<text x="238.76" y="7.62" size="2.54" layer="91">V2.3</text>
 </plain>
 <instances>
