File: Brakeman_array.brd (EAGLE design)
At the start: 99.2 x 71.8 mm, 72 parts

Commit message: 2.1
Parts:
- removed PADN1, PADN10, PADN11, PADN12, PADN13, PADN14, PADN15, PADN16, PADN17, PADN18, PADN19, PADN2, PADN20, PADN21, PADN22, PADN23, PADN24, PADN25, PADN26, PADN27, PADN28, PADN29, PADN3, PADN30, PADN31, PADN32, PADN4, PADN5, PADN6, PADN7, PADN8, PADN9, PADS1, PADS10, PADS11, PADS12, PADS13, PADS14, PADS15, PADS16, PADS2, PADS3, PADS4, PADS5, PADS6, PADS7, PADS8, PADS9: (no value), wirepad:SMD1.27-2.54
- added PADNA, PADNA1, PADNA10, PADNA11, PADNA12, PADNA13, PADNA14, PADNA15, PADNA2, PADNA3, PADNA4, PADNA5, PADNA6, PADNA7, PADNA8, PADNA9, PADNF, PADNF1, PADNF10, PADNF11, PADNF12, PADNF13, PADNF14, PADNF15, PADNF2, PADNF3, PADNF4, PADNF5, PADNF6, PADNF7, PADNF8, PADNF9, PADSF, PADSF1, PADSF10, PADSF11, PADSF12, PADSF13, PADSF14, PADSF15, PADSF2, PADSF3, PADSF4, PADSF5, PADSF6, PADSF7, PADSF8, PADSF9: (no value), wirepad:SMD1.27-2.54
- moved PADL16 101.7 mm to (83.3, 78.4), turned to 70 degrees
- moved R8 97.0 mm to (87.0, 71.5), turned to 90 degrees
- moved PADL15 95.7 mm to (90.8, 65.2), turned to 270 degrees
- moved PADL12 76.9 mm to (57.9, 78.4), turned to 70 degrees
- moved PADL6 71.5 mm to (42.2, 1.65), turned to 250 degrees
- moved R6 62.9 mm to (61.6, 71.5), turned to 90 degrees
- moved R3 60.6 mm to (38.5, 8.51), turned to 270 degrees
- moved PADL1 56.6 mm to (16.8, 1.65), turned to 250 degrees
- moved PADL2 56.5 mm to (9.27, 14.9), turned to 90 degrees
- moved R1 56.3 mm to (13.1, 8.51), turned to 270 degrees
- moved PADL5 53.0 mm to (34.7, 14.9), turned to 90 degrees
- moved PADL8 51.5 mm to (32.5, 78.4)
- moved PADL14 51.5 mm to (93.0, 1.65)
- moved PADL7 51.0 mm to (40.0, 65.2)
- moved PADL13 51.0 mm to (85.5, 14.9)
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Connections:
- new net N: PADNA.1, PADNA2.1, PADNF.1, PADNF2.1
- new net N1: PADNA1.1, PADNA3.1, PADNF1.1, PADNF3.1
- new net N2: PADNA4.1, PADNA5.1, PADNF4.1, PADNF5.1
- new net N3: PADNA6.1, PADNA7.1, PADNF6.1, PADNF7.1
- new net N4: PADNA8.1, PADNA9.1, PADNF8.1, PADNF9.1
- new net N5: PADNA10.1, PADNA11.1, PADNF10.1, PADNF11.1
- new net N6: PADNA12.1, PADNA13.1, PADNF12.1, PADNF13.1
- new net N7: PADNA14.1, PADNA15.1, PADNF14.1, PADNF15.1
- net S: now also PADSF.1, PADSF2.1; no longer PADN2.1, PADN3.1, PADN4.1, PADN6.1, PADS2.1, PADS4.1
- net S1: now also PADSF1.1, PADSF3.1; no longer PADN1.1, PADN5.1, PADN7.1, PADN8.1, PADS1.1, PADS3.1
- net S2: now also PADSF4.1, PADSF5.1; no longer PADN10.1, PADN11.1, PADN12.1, PADN9.1, PADS5.1, PADS6.1
- net S3: now also PADSF6.1, PADSF7.1; no longer PADN13.1, PADN14.1, PADN15.1, PADN16.1, PADS7.1, PADS8.1
- net S4: now also PADSF8.1, PADSF9.1; no longer PADN17.1, PADN18.1, PADN19.1, PADN20.1, PADS10.1, PADS9.1
- net S5: now also PADSF10.1, PADSF11.1; no longer PADN21.1, PADN22.1, PADN23.1, PADN24.1, PADS11.1, PADS12.1
- net S6: now also PADSF12.1, PADSF13.1; no longer PADN25.1, PADN26.1, PADN27.1, PADN28.1, PADS13.1, PADS14.1
- net S7: now also PADSF14.1, PADSF15.1; no longer PADN29.1, PADN30.1, PADN31.1, PADN32.1, PADS15.1, PADS16.1
Routing:
- net N4: track 0.00 -> 62.7 mm, vias 0 -> 3
- net N: track 0.00 -> 62.7 mm, vias 0 -> 3
- net N2: track 0.00 -> 62.7 mm, vias 0 -> 3
- net N6: track 0.00 -> 62.7 mm, vias 0 -> 3
- net N7: track 0.00 -> 62.6 mm, vias 0 -> 3
- net N5: track 0.00 -> 62.6 mm, vias 0 -> 3
- net N1: track 0.00 -> 62.6 mm, vias 0 -> 3
- net N3: track 0.00 -> 62.6 mm, vias 0 -> 3
- net S1: track 43.5 -> 51.6 mm, vias 4 -> 2
- net S5: track 43.5 -> 51.6 mm, vias 4 -> 2
- net S3: track 43.5 -> 51.6 mm, vias 4 -> 2
- net S7: track 43.5 -> 51.6 mm, vias 4 -> 2
- net S2: track 43.5 -> 51.5 mm, vias 4 -> 2
- net S4: track 43.5 -> 51.5 mm, vias 4 -> 2
- net S: track 43.5 -> 51.5 mm, vias 4 -> 2
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- added copper zone on layer 1, net N
- added copper zone on layer 16, net N
- added copper zone on layer 1, net N1
- added copper zone on layer 16, net N1
- added copper zone on layer 1, net N2
- added copper zone on layer 16, net N2
- added copper zone on layer 1, net N3
- added copper zone on layer 16, net N3
- added copper zone on layer 1, net N4
- added copper zone on layer 16, net N4
- added copper zone on layer 1, net N5
- added copper zone on layer 16, net N5
- added copper zone on layer 1, net N6
- added copper zone on layer 16, net N6
- added copper zone on layer 1, net N7
- added copper zone on layer 16, net N7
- added copper zone on layer 1, net S
- added copper zone on layer 1, net S1
- added copper zone on layer 1, net S2
- added copper zone on layer 1, net S3
- added copper zone on layer 1, net S4
- added copper zone on layer 1, net S5
- added copper zone on layer 1, net S6
- added copper zone on layer 1, net S7
Other:
- board size 99.2 x 71.8 mm -> 106.7 x 82.5 mm
- board text added: "DCC Flagman"
- board text added: "V-Score"
- board text removed: "DCC Flagman & Fusee"

Commit message: 2.2
Parts:
- moved PADNF8 51.8 mm to (73.7, 63.3)
- moved PADL10 51.8 mm to (67.2, 53.5)
- moved PADL9 51.8 mm to (59.7, 66.7)
- moved PADNA8 51.8 mm to (59.7, 66.7)
- moved PADNA9 51.8 mm to (67.2, 53.5)
- moved PADNF9 51.8 mm to (73.7, 63.3)
- moved PADSF8 51.8 mm to (73.6, 57.1)
- moved PADSF9 51.8 mm to (73.7, 57.1)
- moved R5 51.8 mm to (63.5, 60.3)
- moved PADNF 51.8 mm to (23.0, 63.3)
- moved PADL1 51.8 mm to (16.5, 53.5)
- moved PADL2 51.8 mm to (9.04, 66.7)
- moved PADNA 51.8 mm to (16.5, 53.5)
- moved PADNA2 51.8 mm to (9.04, 66.7)
- moved PADNF2 51.8 mm to (23.0, 63.3)
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Other:
- board size 106.7 x 82.5 mm -> 106.8 x 106.7 mm
- board text added: "V-Groove 6x places horizontal 6x places vertical"
- board text removed: "V-Score"

Commit message: 2.3
Parts:
- moved PADL5 47.1 mm to (42.1, 79.4), turned to 0 degrees
- moved PADNA4 47.1 mm to (42.1, 79.4), turned to 0 degrees
- moved PADL13 47.1 mm to (89.9, 79.4), turned to 0 degrees
- moved PADNA12 47.1 mm to (89.9, 79.4), turned to 0 degrees
- moved PADNF11 45.6 mm to (62.6, 20.0), flipped to the bottom, turned to 270 degrees
- moved PADNF10 45.6 mm to (62.6, 20.0), flipped to the top, turned to 90 degrees
- moved PADNF3 44.8 mm to (14.9, 20.0), flipped to the bottom, turned to 270 degrees
- moved PADNF1 44.7 mm to (14.9, 20.0), flipped to the top, turned to 90 degrees
- moved PADSF11 42.3 mm to (56.5, 20.0), flipped to the bottom, turned to 270 degrees
- moved PADSF10 42.3 mm to (56.5, 20.0), flipped to the top, turned to 90 degrees
- moved PADL11 41.2 mm to (66.0, 33.7), flipped to the top, turned to 0 degrees
- moved PADNA10 41.2 mm to (66.0, 33.7), flipped to the bottom, turned to 0 degrees
- moved PADSF3 41.0 mm to (8.71, 20.0), flipped to the bottom, turned to 270 degrees
- moved PADSF1 41.0 mm to (8.71, 20.0), flipped to the top, turned to 90 degrees
- moved R6 40.8 mm to (59.7, 29.8), flipped to the bottom, turned to 0 degrees
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Routing:
- net S3: track 51.5 -> 19.7 mm
- net S2: track 51.5 -> 19.7 mm
- net S1: track 51.5 -> 19.7 mm
- net S: track 51.5 -> 19.7 mm
- net S4: track 51.5 -> 19.7 mm
- net S7: track 51.5 -> 19.7 mm
- net S5: track 51.5 -> 19.7 mm
- net S6: track 51.5 -> 19.7 mm
- net N5: track 62.7 -> 38.6 mm, vias 3 -> 2
- net N7: track 62.7 -> 38.6 mm, vias 3 -> 2
- net N6: track 62.7 -> 38.6 mm, vias 3 -> 2
- net N3: track 62.7 -> 38.6 mm, vias 3 -> 2
- net N1: track 62.7 -> 38.6 mm, vias 3 -> 2
- net N4: track 62.7 -> 38.6 mm, vias 3 -> 2
- net N2: track 62.7 -> 38.6 mm, vias 3 -> 2
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Other:
- board size 106.8 x 106.7 mm -> 105.4 x 98.6 mm
- board text added: "2016.11"
- board text added: "Break off and discard"
- board text added: "Safety Sam"
- board text added: "V-Groove"
- board text added: "V2.3"
- board text removed: "2016.04"
- board text removed: "V-Groove 6x places horizontal 6x places vertical"

Commit message: added values for connectors
Parts:
- PADL1, PADL10, PADL11, PADL12, PADL13, PADL14, PADL15, PADL16, PADL2, PADL3, PADL4, PADL5, PADL6, PADL7, PADL8, PADL9, PADNF, PADNF1, PADNF10, PADNF12, PADNF14, PADNF4, PADNF6, PADNF8, PADSF, PADSF1, PADSF10, PADSF12, PADSF14, PADSF4, PADSF6, PADSF8: value (none) -> pad

Commit message: added values for connectors
Parts:
- PADNA, PADNA1, PADNA10, PADNA11, PADNA12, PADNA13, PADNA14, PADNA15, PADNA2, PADNA3, PADNA4, PADNA5, PADNA6, PADNA7, PADNA8, PADNA9, PADNF11, PADNF13, PADNF15, PADNF2, PADNF3, PADNF5, PADNF7, PADNF9, PADSF11, PADSF13, PADSF15, PADSF2, PADSF3, PADSF5, PADSF7, PADSF9: value (none) -> pad

Commit message: Version 2.4
Parts:
- removed PADL1, PADL10, PADL11, PADL12, PADL13, PADL14, PADL15, PADL16, PADL2, PADL3, PADL4, PADL5, PADL6, PADL7, PADL8, PADL9, PADNA, PADNA1, PADNA10, PADNA11, PADNA12, PADNA13, PADNA14, PADNA15, PADNA2, PADNA3, PADNA4, PADNA5, PADNA6, PADNA7, PADNA8, PADNA9, PADNF, PADNF1, PADNF10, PADNF11, PADNF12, PADNF13, PADNF14, PADNF15, PADNF2, PADNF3, PADNF4, PADNF5, PADNF6, PADNF7, PADNF8, PADNF9, PADSF, PADSF1, PADSF10, PADSF11, PADSF12, PADSF13, PADSF14, PADSF15, PADSF2, PADSF3, PADSF4, PADSF5, PADSF6, PADSF7, PADSF8, PADSF9: pad, wirepad:SMD1.27-2.54
- removed R1, R2, R3, R4, R5, R6, R7, R8: 1k0, resistor:0204/5
- added LED1X11, LED1X12, LED1X21, LED1X22, LED1X31, LED1X32, LED1X41, LED1X42, LED2X11, LED2X12, LED2X21, LED2X22, LED2X31, LED2X32, LED2X41, LED2X42: (no value), SPCoast:0603-LED
- added PADNF1X11, PADNF1X12, PADNF1X21, PADNF1X22, PADNF1X31, PADNF1X32, PADNF1X41, PADNF1X42, PADNFX11, PADNFX12, PADNFX21, PADNFX22, PADNFX31, PADNFX32, PADNFX41, PADNFX42, PADSF1X11, PADSF1X12, PADSF1X21, PADSF1X22, PADSF1X31, PADSF1X32, PADSF1X41, PADSF1X42, PADSFX11, PADSFX12, PADSFX21, PADSFX22, PADSFX31, PADSFX32, PADSFX41, PADSFX42: pad, SPCoast:SMD1,27-2,54
- added R1KX11, R1KX12, R1KX21, R1KX22, R1KX31, R1KX32, R1KX41, R1KX42: 1k0, resistor:R0603
Connections:
- removed net LIMITED: PADL1.1, PADL2.1, R1.1
- removed net LIMITED1: PADL3.1, PADL4.1, R2.1
- removed net LIMITED2: PADL5.1, PADL6.1, R3.1
- removed net LIMITED3: PADL7.1, PADL8.1, R4.1
- removed net LIMITED4: PADL10.1, PADL9.1, R5.1
- removed net LIMITED5: PADL11.1, PADL12.1, R6.1
- removed net LIMITED6: PADL13.1, PADL14.1, R7.1
- removed net LIMITED7: PADL15.1, PADL16.1, R8.1
- removed net N: PADNA.1, PADNA2.1, PADNF.1, PADNF2.1
- removed net N1: PADNA1.1, PADNA3.1, PADNF1.1, PADNF3.1
- removed net N2: PADNA4.1, PADNA5.1, PADNF4.1, PADNF5.1
- removed net N3: PADNA6.1, PADNA7.1, PADNF6.1, PADNF7.1
- removed net N4: PADNA8.1, PADNA9.1, PADNF8.1, PADNF9.1
- removed net N5: PADNA10.1, PADNA11.1, PADNF10.1, PADNF11.1
- removed net N6: PADNA12.1, PADNA13.1, PADNF12.1, PADNF13.1
- removed net N7: PADNA14.1, PADNA15.1, PADNF14.1, PADNF15.1
- removed net S: PADSF.1, PADSF2.1, R1.2
- removed net S1: PADSF1.1, PADSF3.1, R2.2
- removed net S2: PADSF4.1, PADSF5.1, R3.2
- removed net S3: PADSF6.1, PADSF7.1, R4.2
- removed net S4: PADSF8.1, PADSF9.1, R5.2
- removed net S5: PADSF10.1, PADSF11.1, R6.2
- removed net S6: PADSF12.1, PADSF13.1, R7.2
- removed net S7: PADSF14.1, PADSF15.1, R8.2
- new net LIMITEDX11: LED1X11.C, LED2X11.A, R1KX11.1
- new net LIMITEDX12: LED1X12.C, LED2X12.A, R1KX12.1
- new net LIMITEDX21: LED1X21.C, LED2X21.A, R1KX21.1
- new net LIMITEDX22: LED1X22.C, LED2X22.A, R1KX22.1
- new net LIMITEDX31: LED1X31.C, LED2X31.A, R1KX31.1
- new net LIMITEDX32: LED1X32.C, LED2X32.A, R1KX32.1
- new net LIMITEDX41: LED1X41.C, LED2X41.A, R1KX41.1
- new net LIMITEDX42: LED1X42.C, LED2X42.A, R1KX42.1
- new net NX11: LED1X11.A, LED2X11.C, PADNF1X11.1, PADNFX11.1
- new net NX12: LED1X12.A, LED2X12.C, PADNF1X12.1, PADNFX12.1
- new net NX21: LED1X21.A, LED2X21.C, PADNF1X21.1, PADNFX21.1
- new net NX22: LED1X22.A, LED2X22.C, PADNF1X22.1, PADNFX22.1
- new net NX31: LED1X31.A, LED2X31.C, PADNF1X31.1, PADNFX31.1
- new net NX32: LED1X32.A, LED2X32.C, PADNF1X32.1, PADNFX32.1
- new net NX41: LED1X41.A, LED2X41.C, PADNF1X41.1, PADNFX41.1
- new net NX42: LED1X42.A, LED2X42.C, PADNF1X42.1, PADNFX42.1
- new net SX11: PADSF1X11.1, PADSFX11.1, R1KX11.2
- new net SX12: PADSF1X12.1, PADSFX12.1, R1KX12.2
- new net SX21: PADSF1X21.1, PADSFX21.1, R1KX21.2
- new net SX22: PADSF1X22.1, PADSFX22.1, R1KX22.2
- new net SX31: PADSF1X31.1, PADSFX31.1, R1KX31.2
- new net SX32: PADSF1X32.1, PADSFX32.1, R1KX32.2
- new net SX41: PADSF1X41.1, PADSFX41.1, R1KX41.2
- new net SX42: PADSF1X42.1, PADSFX42.1, R1KX42.2
Routing:
- net N: track 38.6 -> 0.00 mm, vias 2 -> 0
- net N2: track 38.6 -> 0.00 mm, vias 2 -> 0
- net N4: track 38.6 -> 0.00 mm, vias 2 -> 0
- net N6: track 38.6 -> 0.00 mm, vias 2 -> 0
- net N1: track 38.6 -> 0.00 mm, vias 2 -> 0
- net N3: track 38.6 -> 0.00 mm, vias 2 -> 0
- net N5: track 38.6 -> 0.00 mm, vias 2 -> 0
- net N7: track 38.6 -> 0.00 mm, vias 2 -> 0
- net NX42: track 0.00 -> 35.5 mm, vias 0 -> 4
- net NX32: track 0.00 -> 35.5 mm, vias 0 -> 4
- net NX22: track 0.00 -> 35.5 mm, vias 0 -> 4
- net NX12: track 0.00 -> 35.5 mm, vias 0 -> 4
- net NX41: track 0.00 -> 35.5 mm, vias 0 -> 4
- net NX31: track 0.00 -> 35.5 mm, vias 0 -> 4
- net NX21: track 0.00 -> 35.5 mm, vias 0 -> 4
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- added copper zone on layer 1, net NX11
- added copper zone on layer 16, net NX11
- added copper zone on layer 1, net NX12
- added copper zone on layer 16, net NX12
- added copper zone on layer 1, net NX21
- added copper zone on layer 16, net NX21
- added copper zone on layer 1, net NX22
- added copper zone on layer 16, net NX22
- added copper zone on layer 1, net NX31
- added copper zone on layer 16, net NX31
- added copper zone on layer 1, net NX32
- added copper zone on layer 16, net NX32
- added copper zone on layer 1, net NX41
- added copper zone on layer 16, net NX41
- added copper zone on layer 1, net NX42
- added copper zone on layer 16, net NX42
- added copper zone on layer 1, net SX11
- added copper zone on layer 16, net SX11
- added copper zone on layer 1, net SX12
- added copper zone on layer 16, net SX12
- added copper zone on layer 1, net SX21
- added copper zone on layer 16, net SX21
- added copper zone on layer 1, net SX22
- added copper zone on layer 16, net SX22
- added copper zone on layer 1, net SX31
- added copper zone on layer 16, net SX31
- added copper zone on layer 1, net SX32
- added copper zone on layer 16, net SX32
- added copper zone on layer 1, net SX41
- added copper zone on layer 16, net SX41
- added copper zone on layer 1, net SX42
- added copper zone on layer 16, net SX42
- removed copper zone on layer 1, net N
- removed copper zone on layer 16, net N
- removed copper zone on layer 1, net N1
- removed copper zone on layer 16, net N1
- removed copper zone on layer 1, net N2
- removed copper zone on layer 16, net N2
- removed copper zone on layer 1, net N3
- removed copper zone on layer 16, net N3
- removed copper zone on layer 1, net N4
- removed copper zone on layer 16, net N4
- removed copper zone on layer 1, net N5
- removed copper zone on layer 16, net N5
- removed copper zone on layer 1, net N6
- removed copper zone on layer 16, net N6
- removed copper zone on layer 1, net N7
- removed copper zone on layer 16, net N7
- removed copper zone on layer 1, net S
- removed copper zone on layer 16, net S
- removed copper zone on layer 1, net S1
- removed copper zone on layer 16, net S1
- removed copper zone on layer 1, net S2
- removed copper zone on layer 16, net S2
- removed copper zone on layer 1, net S3
- removed copper zone on layer 16, net S3
- removed copper zone on layer 1, net S4
- removed copper zone on layer 16, net S4
- removed copper zone on layer 1, net S5
- removed copper zone on layer 16, net S5
- removed copper zone on layer 1, net S6
- removed copper zone on layer 16, net S6
- removed copper zone on layer 1, net S7
- removed copper zone on layer 16, net S7
Other:
- board size 105.4 x 98.6 mm -> 103.1 x 99.1 mm
- board text added: "2016.11 2024.01"
- board text added: "John Plocher 2024.01"
- board text added: "Safety Sam DCC Flagman"
- board text added: "V-Score"
- board text removed: "2016.11"
- board text removed: "Break off and discard"
- board text removed: "V-Groove"
- board text removed: "V2.3"
